File: Mensajes_lcd/Mensajes_lcd.kicad_pcb (KiCad board)
At the start: 2 copper layers, 107.9 x 83 mm, 22 parts, among them J1 Conn_01x16_Socket, Q1 MMBT3904, SW1 SW_Push, SW2 SW_Push, SW3 SW_Push, SW4 SW_Push, SW5 SW_Push, SW6 SW_Push, SW7 SW_Push_SPDT, U1 ESP32-C3_SUPERMINI_TH, U2 MT3608

Commit message: Add files via upload
Parts:
- removed RV2: R_Potentiometer_Trim_US, Potentiometer_SMD:Potentiometer_Bourns_3314G_Vertical
- removed the SW7 at (171.1, 63.7)
- added C3: 10M, Capacitor_SMD:C_1206_3216Metric, B.Cu at (165.6, 75.3)
- added C4: C, Capacitor_SMD:C_1206_3216Metric, B.Cu at (150.4, 69.6)
- added C5: C, Capacitor_SMD:C_1206_3216Metric, B.Cu at (160.3, 83.8)
- added C6: C_Polarized, Capacitor_SMD:CP_Elec_3x5.3, B.Cu at (171.7, 86.4)
- added D3: 1N4007, Diode_SMD:D_1206_3216Metric_Pad1.42x1.75mm_HandSolder, B.Cu at (154.4, 83.8)
- added D4: SS34, Diode_SMD:D_SMA, B.Cu at (149.1, 81.5)
- added G***: LOGO, logo:logo_2, B.Cu at (77.7, 86.1)
- added Q1: FS8205A, Package_SO:TSSOP-8_4.4x3mm_P0.65mm, B.Cu at (159.8, 75.8)
- added R1: 1k, Resistor_SMD:R_1206_3216Metric, B.Cu at (165.4, 67.9)
- added R2: 1k, Resistor_SMD:R_1206_3216Metric, B.Cu at (165.5, 71.5)
- added R4: 100, Resistor_SMD:R_1206_3216Metric, B.Cu at (165.5, 79.1)
- added R5: 1k, Resistor_SMD:R_1206_3216Metric, B.Cu at (149.2, 74.9)
- added R8: R, Resistor_SMD:R_1206_3216Metric, B.Cu at (142.7, 78.6)
- added R9: R, Resistor_SMD:R_1206_3216Metric, B.Cu at (142.9, 75.0)
- added SW1: SW_Push_DPDT, Button_Switch_THT:SW_CK_JS202011AQN_DPDT_Angled, F.Cu at (169.6, 79.3)
- added U1: TP4056-42-ESOP8, Package_SO:SOIC-8-1EP_3.9x4.9mm_P1.27mm_EP2.29x3mm, B.Cu at (158.7, 65.8)
- added U3: MT3608, Package_TO_SOT_SMD:SOT-23-6, B.Cu at (155.0, 79.3)
- BT1: value BK-18650-PC4 -> Battery; footprint Componentes_varios:BAT_BK-18650-PC4 -> Battery:BatteryHolder_MPD_BH-18650-PC
- C2: value C -> 0,1mf
- D1: value SM4007 -> Azul; footprint Diode_SMD:D_MELF -> LED_THT:LED_D3.0mm; moved to F.Cu
- D2: value SS34 -> Rojo; footprint Diode_SMD:D_SMA -> LED_THT:LED_D3.0mm; moved to F.Cu
- L1: value AX104R-221 -> L; footprint Inductor_SMD:IND_AX104R-221 -> Inductor_SMD:L_10.4x10.4_H4.8
- R3: value R -> 1,2k
- U2: value MT3608 -> DW01A
- moved BT1 38.0 mm to (169.2, 103.9), turned to 180 degrees
- moved C1 31.1 mm to (154.2, 69.6), turned to 90 degrees
- moved C2 24.6 mm to (165.4, 83.7)
- moved D1 22.5 mm to (171.3, 64.8), turned to 90 degrees
- moved D2 21.1 mm to (171.3, 70.3), turned to 90 degrees
- moved U2 13.7 mm to (154.9, 74.3), turned to 0 degrees
- moved L1 11.9 mm to (142.0, 67.3), turned to 180 degrees
- moved R3 5.11 mm to (154.2, 64.3), turned to -90 degrees
- moved Q2 2.25 mm to (116.4, 74.6)
- moved R7 0.89 mm to (116.9, 70.4)
- renumbered Q1 to Q2, R1 to R6, R2 to R7, SW1 to SW2, SW2 to SW3, SW3 to SW4, SW4 to SW5, SW5 to SW6, SW6 to SW7, U1 to U4
Connections:
- C1 pad 1: Net-(U2-EN) -> +5V-usb
- C2 pad 1: +5V -> Net-(U2-VCC)
- C2 pad 2: GND -> Bat-
- D1 pad 2: VCC -> +5V-usb
- D2 pad 1: +5V -> Net-(D2-K)
- D2 pad 2: Net-(D2-A) -> +5V-usb
- J1 pad 2: VCC -> +5V-conv
- L1 pad 1: Net-(U2-EN) -> Net-(U3-EN)
- L1 pad 2: Net-(D2-A) -> Net-(D4-A)
- R6 pad 2: VCC -> +5V-conv
- RV1 pad 1: VCC -> +5V-conv
- U2 pad 1: Net-(D2-A) -> Net-(U2-OD)
- U2 pad 2: GND -> Net-(U2-CS)
- U2 pad 4: Net-(U2-EN) -> unconnected-(U2-TD-Pad4)
- U2 pad 5: Net-(U2-EN) -> Net-(U2-VCC)
- U2 pad 6: unconnected-(U2-NC-Pad6) -> Bat-
- U4 pad 5V: Net-(D1-K) -> Usb-c
Routing:
- net Usb-c: track 0.00 -> 126.4 mm, vias 0 -> 1
- net Bat-: track 0.00 -> 116.4 mm, vias 0 -> 4
- net VCC: track 115.9 -> 0.00 mm, vias 1 -> 0
- net +5V-conv: track 0.00 -> 110.4 mm, vias 0 -> 1
- net Net-(D1-K): track 95.6 -> 6.00 mm, vias 1 -> 0
- net Net-(U2-EN): track 85.3 -> 0.00 mm, vias 1 -> 0
- net +5V-usb: track 0.00 -> 46.6 mm, vias 0 -> 2
- net Net-(U3-EN): track 0.00 -> 35.7 mm, vias 0 -> 3
- net +5V: track 32.2 -> 0.00 mm
- net Net-(BT1-+): track 0.00 -> 28.9 mm
- net Net-(D4-A): track 0.00 -> 26.2 mm, vias 0 -> 2
- net Net-(D3-K): track 0.00 -> 22.2 mm, vias 0 -> 2
- net Net-(U1-BAT): track 0.00 -> 22.0 mm, vias 0 -> 3
- net Net-(U3-FB): track 0.00 -> 17.3 mm
- net Net-(D2-A): track 17.2 -> 0.00 mm, vias 2 -> 0
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Other:
- outline, holes or cut-outs redrawn
- board text added: "Comunicador para sordos"
