File: Mensajes_lcd/Mensajes_lcd.kicad_sch (KiCad schematic)
At the start: 22 parts, among them J1 Conn_01x16_Socket, Q1 MMBT3904, SW1 SW_Push, SW2 SW_Push, SW3 SW_Push, SW4 SW_Push, SW5 SW_Push, SW6 SW_Push, SW7 SW_Push_SPDT, U1 ESP32-C3_SUPERMINI_TH, U2 MT3608

Commit message: Add files via upload
Parts:
- removed BT1: BK-18650-PC4, Componentes_varios:BAT_BK-18650-PC4, symbol BK-18650-PC4:BK-18650-PC4
- removed D1: SM4007, Diode_SMD:D_MELF, symbol Diode:SM4007
- removed D2: SS34, Diode_SMD:D_SMA, symbol Diode:SS34
- removed L1: AX104R-221, Inductor_SMD:IND_AX104R-221, symbol AX104R-221:AX104R-221
- removed RV2: R_Potentiometer_Trim_US, Potentiometer_SMD:Potentiometer_Bourns_3314G_Vertical, symbol Device:R_Potentiometer_Trim_US
- removed SW7: SW_Push_SPDT, Button_Switch_THT:SW_Slide_SPDT_Straight_CK_OS102011MS2Q, symbol Switch:SW_Push_SPDT
- removed U2: MT3608, Package_TO_SOT_SMD:SOT-23-6, symbol Regulator_Switching:MT3608
- added BT1: Battery, Battery:BatteryHolder_MPD_BH-18650-PC, symbol Device:Battery
- added C3: 10M, Capacitor_SMD:C_1206_3216Metric, symbol Device:C
- added C4, C5: C, Capacitor_SMD:C_1206_3216Metric, symbol Device:C
- added C6: C_Polarized, Capacitor_SMD:CP_Elec_3x5.3, symbol Device:C_Polarized
- added D1: Azul, LED_THT:LED_D3.0mm, symbol Device:LED
- added D2: Rojo, LED_THT:LED_D3.0mm, symbol Device:LED
- added D3: 1N4007, Diode_SMD:D_1206_3216Metric_Pad1.42x1.75mm_HandSolder, symbol Diode:1N4007
- added D4: SS34, Diode_SMD:D_SMA, symbol Diode:SS34
- added L1: L, Inductor_SMD:L_10.4x10.4_H4.8, symbol Device:L
- added Q1: FS8205A, Package_SO:TSSOP-8_4.4x3mm_P0.65mm, symbol FS8205A:FS8205A
- added R1, R2, R5: 1k, Resistor_SMD:R_1206_3216Metric, symbol Device:R
- added R4: 100, Resistor_SMD:R_1206_3216Metric, symbol Device:R
- added R8, R9: R, Resistor_SMD:R_1206_3216Metric, symbol Device:R
- added SW1: SW_Push_DPDT, Button_Switch_THT:SW_CK_JS202011AQN_DPDT_Angled, symbol Switch:SW_Push_DPDT
- added U1: TP4056-42-ESOP8, Package_SO:SOIC-8-1EP_3.9x4.9mm_P1.27mm_EP2.29x3mm, symbol Battery_Management:TP4056-42-ESOP8
- added U2: DW01A, Package_TO_SOT_SMD:SOT-23-6, symbol Battery_Management:DW01A
- added U3: MT3608, Package_TO_SOT_SMD:SOT-23-6, symbol Regulator_Switching:MT3608
- C2: value C -> 0,1mf
- R3: value R -> 1,2k
- renumbered Q1 to Q2, R1 to R6, R2 to R7, SW1 to SW2, SW2 to SW3, SW3 to SW4, SW4 to SW5, SW5 to SW6, SW6 to SW7, U1 to U4
Connections:
- net GND: now also C3.2, C4.2, C5.2, C6.2, Q1.6, Q1.7, R5.2, R9.2, U1.1 (TEMP), U1.3 (GND), U1.9 (EPAD), U3.2 (GND); no longer C2.2
- net at R3.1: now also U1.2 (PROG)
- net Usb-c: now reaches U4.5V
- net Usb-c: now also C6.1, SW1.5 (B)
- net +5V-usb: now reaches C1.1
- net +5V-usb: now also D1.2 (A), D2.2 (A), SW1.4 (A), U1.4 (V_{CC}), U1.8 (CE)
- net +5V: no longer names the net of C2.1
- net +5V: now also R4.1, U2.5 (VCC)
- net VCC renamed +5V-conv
- net +5V-conv: now also C5.1, D3.2 (A), D4.1 (K), R8.1
- new net: D3.1 (K), SW1.6 (C)
- new net: Q1.1, Q1.8
- new net: Q1.4, U2.1 (OD)
- new net: Q1.5, U2.3 (OC)
- new net: D1.1 (K), R1.1
- new net: R8.2, R9.1, U3.3 (FB)
- new net: D4.2 (A), L1.2, U3.1 (SW)
- new net: C4.1, L1.1, SW1.3 (C), U3.4 (EN), U3.5 (IN)
- new net: BT1.1 (+), SW1.2 (B)
- new net: D2.1 (K), R2.1
- new net: R2.2, U1.7 (~{CHRG})
- new net: C3.1, R4.2, SW1.1 (A), U1.5 (BAT)
- new net: R5.1, U2.2 (CS)
- new net: R1.2, U1.6 (~{STDBY})
- new net Bat-: BT1.2 (-), C2.2, Q1.2, Q1.3, U2.6 (GND)
Other:
- moved on the sheet: J1, Q2, R6, R7, RV1, SW2, SW3, SW4, SW5, SW6, SW7, U4
